Commit message: ajout rove_description a jour, fonctionnel sur le jetson

File: src/rove_description/urdf/flipper.urdf.xacro (robot description, xacro)
@@ -75,5 +75,5 @@
                 <origin xyz="0 0 0.5" rpy="0 0 0" />
                 <mass value="1" />
-                <inertia ixx="0" ixy="0" ixz="0" iyy="0" iyz="0" izz="0" />
+                <inertia ixx="0.001042" ixy="0.0" ixz="0.0" iyy="0.013542" iyz="0.0" izz="0.014167" />
             </inertial>
         </link>

File: src/rove_description/urdf/livox.urdf.xacro (robot description, xacro)
@@ -50,4 +50,11 @@
       <child link="${name}_laser"/>
     </joint>
+    <!-- Alias link so the Livox driver's hardcoded 'livox_frame' frame_id resolves in TF -->
+    <link name="livox_frame"/>
+    <joint name="livox_frame_alias_joint" type="fixed">
+      <origin xyz="0 0 0" rpy="0 0 0"/>
+      <parent link="${name}_link"/>
+      <child link="livox_frame"/>
+    </joint>
     <xacro:property name="samples_h" value="${floor((max_ang_h - min_ang_h) * 180 / (ang_res_h * pi) + 0.5)}"/>
     <xacro:property name="samples_v" value="${floor((max_ang_v - min_ang_v) * 180 / (ang_res_v * pi) + 0.5)}"/>

File: src/rove_description/urdf/sensor.urdf.xacro (robot description, xacro)
@@ -10,7 +10,8 @@
     <link name="top_link">
     </link>
+    <!-- IMU (VectorNav VN-300) -->
     <joint name="imu_joint" type="fixed">
         <parent link="top_link" />
-        <child link="camera_link" />
+        <child link="imu_link" />
         <origin xyz="-0.05 0.15 -0.06" rpy="0 0 0" />
     </joint>
@@ -31,4 +32,5 @@
         </collision>
     </link>
+    <!-- Camera -->
     <joint name="camera_joint" type="fixed">
         <parent link="top_link" />
@@ -53,5 +55,5 @@
     </link>
     <xacro:livox_lidar name="livox" parent_link="top_link">
-        <origin xyz="-0.3 0.0 0.13" rpy="0.5235987755983  0 ${-pi/2}" />
+        <origin xyz="-0.3 0.0 0.13" rpy="0  0.5235987755983 ${-pi/2}" />
     </xacro:livox_lidar>
 </robot>
