Commit message: first functionning 2d map

File: src/rove_description/urdf/sensor.urdf.xacro (robot description, xacro)
@@ -55,5 +55,5 @@
     </link>
     <xacro:livox_lidar name="livox" parent_link="top_link">
-        <origin xyz="-0.3 0.0 0.13" rpy="0  0.5235987755983 ${-pi/2}" />
+        <origin xyz="-0.3 0.0 0.13" rpy="0  ${30*(pi/180)} ${pi}" />
     </xacro:livox_lidar>
 </robot>

Commit message: costmap plus fonctionelle

File: src/rove_description/urdf/sensor.urdf.xacro (robot description, xacro)
@@ -14,5 +14,5 @@
         <parent link="top_link" />
         <child link="imu_link" />
-        <origin xyz="-0.05 0.15 -0.06" rpy="0 0 0" />
+        <origin xyz="-0.05 -0.15 -0.06" rpy="0 0 0" />
     </joint>
     <link name="imu_link">
