Commit message: multi-camera support, tf positions still to fix

File: src/rove_description/urdf/rove_standard.urdf (robot description, URDF)
Before this commit: robot rove_standard, 54 links, 53 joints
Links:
- removed link chinese_camera_2_optical_frame
- removed link chinese_camera_3_optical_frame
- removed link chinese_camera_4_optical_frame
- removed link chinese_camera_optical_frame
- added link cam_east_optical_frame
- added link cam_north_optical_frame
- added link cam_south_optical_frame
- added link cam_west_optical_frame
Joints:
- joint chinese_camera_2_optical_joint: child chinese_camera_2_optical_frame -> cam_east_optical_frame
- joint chinese_camera_3_optical_joint: child chinese_camera_3_optical_frame -> cam_south_optical_frame
- joint chinese_camera_4_optical_joint: child chinese_camera_4_optical_frame -> cam_west_optical_frame
- joint chinese_camera_optical_joint: child chinese_camera_optical_frame -> cam_north_optical_frame

Commit message: ajout des cameras alignées aux transforms

File: src/rove_description/urdf/rove_standard.urdf (robot description, URDF)
Before this commit: robot rove_standard, 54 links, 53 joints
Joints:
- joint chinese_camera_2_optical_joint: origin xyz=0 0 0 rpy=-1.5708 0 -1.5708 -> xyz=0 0 0.1 rpy=0 0 0; parent chinese_camera_2 -> chinese_camera
- joint chinese_camera_3_optical_joint: origin xyz=0 0 0 rpy=-1.5708 0 -1.5708 -> xyz=0 0 0.1 rpy=0 0 0; parent chinese_camera_3 -> chinese_camera_4
- joint chinese_camera_4_optical_joint: origin xyz=0 0 0 rpy=-1.5708 0 -1.5708 -> xyz=0 0 0.1 rpy=0 0 0; parent chinese_camera_4 -> chinese_camera_3
- joint chinese_camera_optical_joint: origin xyz=0 0 0 rpy=-1.5708 0 -1.5708 -> xyz=0 0 0.1 rpy=0 0 0; parent chinese_camera -> chinese_camera_2

Commit message: fix 90 degree rotate

File: src/rove_description/urdf/rove_standard.urdf (robot description, URDF)
Before this commit: robot rove_standard, 54 links, 53 joints
Links:
- removed link ASection_pivot
- removed link BSection_pivot
- removed link Base_pivot
- removed link DrumBL_pivot
- removed link DrumBR_pivot
- removed link DrumFL_pivot
- removed link DrumFR_pivot
- removed link FlipperBL_pivot
- removed link FlipperBR_pivot
- removed link FlipperFL_pivot
- removed link FlipperFR_pivot
- removed link JointA_pivot
- removed link JointB_pivot
- removed link JointGripper_pivot
- removed link chinese_camera_2_pivot
- removed link chinese_camera_3_pivot
- removed link chinese_camera_4_pivot
- removed link chinese_camera_5_pivot
- removed link chinese_camera_6_pivot
- removed link chinese_camera_7_pivot
- removed link chinese_camera_pivot
- removed link dji_mid360_2_pivot
- removed link dji_mid360_pivot
- removed link pole_pivot
- added link arm_base_pivot
- added link arm_elbow_pivot
- added link arm_forearm_pivot
- added link arm_gripper_pivot
- added link arm_shoulder_pivot
- added link arm_wrist_pivot
- added link cam_body_front_pivot
- added link cam_body_rear_pivot
- added link cam_east_pivot
- added link cam_gripper_pivot
- added link cam_north_pivot
- added link cam_south_pivot
- added link cam_west_pivot
- added link drum_bl_pivot
- added link drum_br_pivot
- added link drum_fl_pivot
- added link drum_fr_pivot
- added link flipper_bl_pivot
- added link flipper_br_pivot
- added link flipper_fl_pivot
- added link flipper_fr_pivot
- added link lidar_lower_pivot
- added link lidar_upper_pivot
- added link sensor_pole_pivot
Joints:
- removed joint chinese_camera_2_optical_joint
- removed joint chinese_camera_3_optical_joint
- removed joint chinese_camera_4_optical_joint
- removed joint chinese_camera_optical_joint
- removed joint joint_revolute
- removed joint joint_revolute_10
- removed joint joint_revolute_10_offset
- removed joint joint_revolute_11
- removed joint joint_revolute_11_offset
- removed joint joint_revolute_12
- removed joint joint_revolute_12_offset
- removed joint joint_revolute_13
- removed joint joint_revolute_13_offset
- removed joint joint_revolute_14
- removed joint joint_revolute_14_offset
- removed joint joint_revolute_15
- removed joint joint_revolute_15_offset
- removed joint joint_revolute_16
- removed joint joint_revolute_16_offset
- removed joint joint_revolute_17
- removed joint joint_revolute_17_offset
- removed joint joint_revolute_18
- removed joint joint_revolute_18_offset
- removed joint joint_revolute_19
- removed joint joint_revolute_19_offset
- removed joint joint_revolute_2
- removed joint joint_revolute_20
- removed joint joint_revolute_20_offset
- removed joint joint_revolute_21
- removed joint joint_revolute_21_offset
- removed joint joint_revolute_22
- removed joint joint_revolute_22_offset
- removed joint joint_revolute_23
- removed joint joint_revolute_23_offset
- removed joint joint_revolute_24
- removed joint joint_revolute_24_offset
- removed joint joint_revolute_2_offset
- removed joint joint_revolute_3
- removed joint joint_revolute_3_offset
- removed joint joint_revolute_4
- removed joint joint_revolute_4_offset
- removed joint joint_revolute_5
- removed joint joint_revolute_5_offset
- removed joint joint_revolute_6
- removed joint joint_revolute_6_offset
- removed joint joint_revolute_7
- removed joint joint_revolute_7_offset
- removed joint joint_revolute_8
- removed joint joint_revolute_8_offset
- removed joint joint_revolute_9
- removed joint joint_revolute_9_offset
- removed joint joint_revolute_offset
- removed joint vn300_joint
- added joint arm_base_offset: type fixed, parent arm_base_pivot, child Base, origin xyz=0.399414 -0.209923 -0.15 rpy=0 0 0
- added joint arm_base_yaw_joint: type revolute, parent Core, child arm_base_pivot, origin xyz=-0.399414 0.209923 0.221123 rpy=0 0 0, axis 0 0 1, limit lower=-3.14159 upper=3.14159 effort=10 velocity=1
- added joint arm_elbow_offset: type fixed, parent arm_elbow_pivot, child JointA, origin xyz=0.7 -0.255 -0.378 rpy=0 0 0
- added joint arm_elbow_pitch_joint: type revolute, parent ASection, child arm_elbow_pivot, origin xyz=-0.7 0.255 0.378 rpy=0 0 0, axis 0 -1 0, limit lower=-3.14159 upper=3.14159 effort=10 velocity=1
- added joint arm_forearm_offset: type fixed, parent arm_forearm_pivot, child BSection, origin xyz=0.767647 -0.205 -0.378 rpy=0 0 0
- added joint arm_forearm_roll_joint: type revolute, parent JointA, child arm_forearm_pivot, origin xyz=-0.767647 0.205 0.378 rpy=0 0 0, axis -1 0 0, limit lower=-3.14159 upper=3.14159 effort=10 velocity=1
- added joint arm_gripper_offset: type fixed, parent arm_gripper_pivot, child JointGripper, origin xyz=1.1728 -0.20415 -0.378 rpy=0 0 0
- added joint arm_gripper_roll_joint: type revolute, parent JointB, child arm_gripper_pivot, origin xyz=-1.1728 0.20415 0.378 rpy=0 0 0, axis -1 0 0, limit lower=-3.14159 upper=3.14159 effort=10 velocity=1
- added joint arm_shoulder_offset: type fixed, parent arm_shoulder_pivot, child ASection, origin xyz=0.4 -0.27 -0.388 rpy=0 0 0
- added joint arm_shoulder_pitch_joint: type revolute, parent Base, child arm_shoulder_pivot, origin xyz=-0.4 0.27 0.388 rpy=0 0 0, axis 0 1 0, limit lower=-0.5 upper=3.6 effort=10 velocity=1
- added joint arm_wrist_offset: type fixed, parent arm_wrist_pivot, child JointB, origin xyz=1.08936 -0.205 -0.378 rpy=0 0 0
- added joint arm_wrist_pitch_joint: type revolute, parent BSection, child arm_wrist_pivot, origin xyz=-1.1 0.205 0.378 rpy=0 0 0, axis 0 1 0, limit lower=-1.6 upper=1.6 effort=10 velocity=1
- added joint cam_body_front_joint: type fixed, parent Core, child cam_body_front_pivot, origin xyz=0.31746 0.209 0.192576 rpy=0 0 0, axis 1 0 0, limit lower=-3.14159 upper=3.14159 effort=10 velocity=1
- added joint cam_body_front_offset: type fixed, parent cam_body_front_pivot, child chinese_camera_6, origin xyz=0.031733 -0.000947911 -0.0166233 rpy=-1.5708 5.55112e-17 1.5708
- added joint cam_body_rear_joint: type fixed, parent Core, child cam_body_rear_pivot, origin xyz=-0.447106 0.216081 0.168303 rpy=0 0 0, axis -0.999548 0.0300528 0, limit lower=-3.14159 upper=3.14159 effort=10 velocity=1
- added joint cam_body_rear_offset: type fixed, parent cam_body_rear_pivot, child chinese_camera_5, origin xyz=-0.0228113 -0.00141777 -0.0192583 rpy=-1.5708 -5.55112e-17 -1.5708
- added joint cam_east_joint: type revolute, parent pole, child cam_east_pivot, origin xyz=-0.024 -0.0727157 0.587006 rpy=0 0 0, axis 0 -0.46469 0.885474, limit lower=-3.14159 upper=3.14159 effort=10 velocity=1
- added joint cam_east_offset: type fixed, parent cam_east_pivot, child chinese_camera_4, origin xyz=0.0248549 -0.0148706 -0.0090392 rpy=-1.5708 -2.22045e-16 1.60237e-31
- added joint cam_east_optical_joint: type fixed, parent chinese_camera_4, child cam_east_optical_frame, origin xyz=0 0 0.1 rpy=0 0 0
- added joint cam_gripper_joint: type fixed, parent JointGripper, child cam_gripper_pivot, origin xyz=-1.1936 0.205 0.4155 rpy=0 0 0, axis 0 -0.111961 0.993713, limit lower=-3.14159 upper=3.14159 effort=10 velocity=1
- added joint cam_gripper_offset: type fixed, parent cam_gripper_pivot, child chinese_camera_7, origin xyz=0.00311921 6.66671e-05 0.0217355 rpy=-1.5708 -5.55112e-17 -1.5708
- added joint cam_north_joint: type fixed, parent pole, child cam_north_pivot, origin xyz=0.0725343 -0.024 0.587101 rpy=0 0 0, axis 0 1 0, limit lower=-3.14159 upper=3.14159 effort=10 velocity=1
- added joint cam_north_offset: type fixed, parent cam_north_pivot, child chinese_camera, origin xyz=0.0154955 0.0243019 -0.00922952 rpy=-1.5708 0 1.5708
- added joint cam_north_optical_joint: type fixed, parent chinese_camera, child cam_north_optical_frame, origin xyz=0 0 0.1 rpy=0 0 0
- added joint cam_south_joint: type fixed, parent pole, child cam_south_pivot, origin xyz=-0.0730961 0.024 0.586861 rpy=0 0 0, axis 0 -1 0, limit lower=-3.14159 upper=3.14159 effort=10 velocity=1
- added joint cam_south_offset: type fixed, parent cam_south_pivot, child chinese_camera_3, origin xyz=-0.0149206 -0.0234735 -0.00886397 rpy=-1.5708 5.55112e-17 -1.5708
- added joint cam_south_optical_joint: type fixed, parent chinese_camera_3, child cam_south_optical_frame, origin xyz=0 0 0.1 rpy=0 0 0
- added joint cam_west_joint: type fixed, parent pole, child cam_west_pivot, origin xyz=0.024 0.0730961 0.586861 rpy=0 0 0, axis 0 0.23939 0.970923, limit lower=-3.14159 upper=3.14159 effort=10 velocity=1
- added joint cam_west_offset: type fixed, parent cam_west_pivot, child chinese_camera_2, origin xyz=-0.0239323 0.014361 -0.00867528 rpy=-1.5708 -1.38778e-16 3.14159
- added joint cam_west_optical_joint: type fixed, parent chinese_camera_2, child cam_west_optical_frame, origin xyz=0 0 0.1 rpy=0 0 0
- added joint drum_bl_joint: type revolute, parent Core, child drum_bl_pivot, origin xyz=0.290223 0.149 0.0888089 rpy=0 0 0, axis 0 -1 0, limit lower=-3.14159 upper=3.14159 effort=10 velocity=1
- added joint drum_bl_offset: type fixed, parent drum_bl_pivot, child DrumBL, origin xyz=-0.290223 -0.149 -0.0888089 rpy=0 0 0
- added joint drum_br_joint: type revolute, parent Core, child drum_br_pivot, origin xyz=0.290223 0.290223 0.0888089 rpy=0 0 0, axis 0 1 0, limit lower=-3.14159 upper=3.14159 effort=10 velocity=1
- added joint drum_br_offset: type fixed, parent drum_br_pivot, child DrumBR, origin xyz=-0.290223 -0.29 -0.0888089 rpy=0 0 0
- added joint drum_fl_joint: type revolute, parent Core, child drum_fl_pivot, origin xyz=-0.299777 0.149 0.0888089 rpy=0 0 0, axis 0 -1 0, limit lower=-3.14159 upper=3.14159 effort=10 velocity=1
- added joint drum_fl_offset: type fixed, parent drum_fl_pivot, child DrumFL, origin xyz=0.299777 -0.149 -0.0888089 rpy=0 0 0
- added joint drum_fr_joint: type revolute, parent Core, child drum_fr_pivot, origin xyz=-0.299777 0.269 0.0888089 rpy=0 0 0, axis 0 1 0, limit lower=-3.14159 upper=3.14159 effort=10 velocity=1
- added joint drum_fr_offset: type fixed, parent drum_fr_pivot, child DrumFR, origin xyz=0.299777 -0.269 -0.0888089 rpy=0 0 0
- added joint flipper_bl_joint: type revolute, parent Core, child flipper_bl_pivot, origin xyz=0.290223 0 0.0888089 rpy=0 0 0, axis -1.77962e-08 -1 0, limit lower=-3.14159 upper=3.14159 effort=10 velocity=1
- added joint flipper_bl_offset: type fixed, parent flipper_bl_pivot, child FlipperBL, origin xyz=-0.290223 0 -0.0888089 rpy=0 0 0
- added joint flipper_br_joint: type revolute, parent Core, child flipper_br_pivot, origin xyz=0.290223 0.418 0.0888089 rpy=0 0 0, axis 0 1 0, limit lower=-3.14159 upper=3.14159 effort=10 velocity=1
- added joint flipper_br_offset: type fixed, parent flipper_br_pivot, child FlipperBR, origin xyz=-0.290223 -0.418 -0.0888089 rpy=0 0 0
- added joint flipper_fl_joint: type revolute, parent Core, child flipper_fl_pivot, origin xyz=-0.299777 0 0.0888089 rpy=0 0 0, axis 1.77962e-08 -1 0, limit lower=-3.14159 upper=3.14159 effort=10 velocity=1
- added joint flipper_fl_offset: type fixed, parent flipper_fl_pivot, child FlipperFL, origin xyz=0.299777 0 -0.0888089 rpy=0 0 0
- added joint flipper_fr_joint: type revolute, parent Core, child flipper_fr_pivot, origin xyz=-0.299777 0.418 0.0888089 rpy=0 0 0, axis 0 1 0, limit lower=-3.14159 upper=3.14159 effort=10 velocity=1
- added joint flipper_fr_offset: type fixed, parent flipper_fr_pivot, child FlipperFR, origin xyz=0.299777 -0.418 -0.0888089 rpy=0 0 0
- added joint imu_joint: type fixed, parent Core, child vn300_vectornav, origin xyz=0 0 0 rpy=0 0 0
- added joint lidar_lower_joint: type fixed, parent pole, child lidar_lower_pivot, origin xyz=4.59098e-18 0 0.574 rpy=0 0 0, axis 0 0 -1, limit lower=-3.14159 upper=3.14159 effort=10 velocity=1
- added joint lidar_lower_offset: type fixed, parent lidar_lower_pivot, child dji_mid360_2, origin xyz=0.000551953 -0.000521468 -0.0284671 rpy=-1.5708 0 1.5708
- added joint lidar_upper_joint: type fixed, parent pole, child lidar_upper_pivot, origin xyz=-9.31322e-11 -2.66092e-11 0.587 rpy=0 0 0, axis 0 0 1, limit lower=-3.14159 upper=3.14159 effort=10 velocity=1
- added joint lidar_upper_offset: type fixed, parent lidar_upper_pivot, child dji_mid360, origin xyz=0.00112693 0.0015559 0.0289736 rpy=1.5708 0 1.5708
- added joint sensor_pole_joint: type fixed, parent Core, child sensor_pole_pivot, origin xyz=0.31746 0.209 0.221123 rpy=0 0 1.5708, axis 0 0 1, limit lower=-3.14159 upper=3.14159 effort=10 velocity=1
- added joint sensor_pole_offset: type fixed, parent sensor_pole_pivot, child pole, origin xyz=-0.0467844 0.000515604 -0.00281394 rpy=0 0 -1.5708

Commit message: fix urdf mesh + mapping_api + various fixes

File: src/rove_description/urdf/rove_standard.urdf (robot description, URDF)
Before this commit: robot rove_standard, 54 links, 53 joints
Links:
- added link base_link
- added link livox_frame
Joints:
- added joint base_link_to_core: type fixed, parent base_link, child Core, origin xyz=0 0 0 rpy=0 0 0
- added joint livox_frame_joint: type fixed, parent Core, child livox_frame, origin xyz=0.2 0.2 0.7 rpy=0 0 0
- joint cam_body_front_offset: origin xyz=0.031733 -0.000947911 -0.0166233 rpy=-1.5708 5.55112e-17 1.5708 -> xyz=0.031733 -0.000947911 -0.0166233 rpy=-1.5708 0 1.5708
- joint cam_body_rear_offset: origin xyz=-0.0228113 -0.00141777 -0.0192583 rpy=-1.5708 -5.55112e-17 -1.5708 -> xyz=-0.0228113 -0.00141777 -0.0192583 rpy=-1.5708 0 -1.5708
- joint cam_east_offset: origin xyz=0.0248549 -0.0148706 -0.0090392 rpy=-1.5708 -2.22045e-16 1.60237e-31 -> xyz=0.0248549 -0.0148706 -0.0090392 rpy=-1.5708 0 0
- joint cam_gripper_offset: origin xyz=0.00311921 6.66671e-05 0.0217355 rpy=-1.5708 -5.55112e-17 -1.5708 -> xyz=0.00311921 6.66671e-05 0.0217355 rpy=-1.5708 0 -1.5708
- joint cam_south_offset: origin xyz=-0.0149206 -0.0234735 -0.00886397 rpy=-1.5708 5.55112e-17 -1.5708 -> xyz=-0.0149206 -0.0234735 -0.00886397 rpy=-1.5708 0 -1.5708
- joint imu_joint: origin xyz=0 0 0 rpy=0 0 0 -> xyz=0 -0.14 0.06 rpy=-1.5708  0 1.5708

Commit message: reverted fix urdf omfg removed base_link

File: src/rove_description/urdf/rove_standard.urdf (robot description, URDF)
Before this commit: robot rove_standard, 56 links, 55 joints
Joints:
- removed joint base_link_to_core
- added joint core_to_base_link: type fixed, parent Core, child base_link, origin xyz=-0.0386 0.2090 0.1150 rpy=0 0 0
- joint cam_body_front_joint: axis 1 0 0 -> (none); limit lower=-3.14159 upper=3.14159 effort=10 velocity=1 -> (none)
- joint cam_body_rear_joint: axis -0.999548 0.0300528 0 -> (none); limit lower=-3.14159 upper=3.14159 effort=10 velocity=1 -> (none)
- joint cam_gripper_joint: axis 0 -0.111961 0.993713 -> (none); limit lower=-3.14159 upper=3.14159 effort=10 velocity=1 -> (none)
- joint cam_north_joint: axis 0 1 0 -> (none); limit lower=-3.14159 upper=3.14159 effort=10 velocity=1 -> (none)
- joint cam_south_joint: axis 0 -1 0 -> (none); limit lower=-3.14159 upper=3.14159 effort=10 velocity=1 -> (none)
- joint cam_west_joint: axis 0 0.23939 0.970923 -> (none); limit lower=-3.14159 upper=3.14159 effort=10 velocity=1 -> (none)
- joint imu_joint: origin xyz=0 -0.14 0.06 rpy=-1.5708  0 1.5708 -> xyz=0 -0.14 0.06 rpy=-1.5708 0 1.5708
- joint lidar_lower_joint: axis 0 0 -1 -> (none); limit lower=-3.14159 upper=3.14159 effort=10 velocity=1 -> (none)
- joint lidar_upper_joint: axis 0 0 1 -> (none); limit lower=-3.14159 upper=3.14159 effort=10 velocity=1 -> (none)
- joint livox_frame_joint: origin xyz=0.2 0.2 0.7 rpy=0 0 0 -> xyz=0 0 0.581 rpy=0 0 0; parent Core -> pole
- joint sensor_pole_joint: axis 0 0 1 -> (none); limit lower=-3.14159 upper=3.14159 effort=10 velocity=1 -> (none)
