Commit message: rove_sim_webots: real-Rove fidelity + dual-lidar merger
Update the Webots sim to match the rove_standard.urdf hardware (live
2026-06-01 robot_description), with one practical override.

URDF + topics:
- proto: 4 cameras (cam_north/east/south/west) at exact URDF positions
  on the pole, replacing the single rove_camera. Topics + frame names
  match real-bag conventions.
- proto: lidar topics renamed to /livox/lidar_192_168_2_{40,41}; IMU
  to /livox/imu_192_168_2_40 (real-bag names).
- proto: IMU triplet moved to Core (real Rove's VN-300 mount).
- urdf: 4 camera <device> blocks; base_link <- Core anchor so the
  external RSP (driven by rove_standard.urdf) lines up.
- sim.launch.py: new imu_relay /livox/imu_192_168_2_40 -> /imu/data
  so SLAM still receives IMU (until enable_imu_factor is wired).

Mount geometry (verified vs URDF chain):
- TOP lidar upright, BOTTOM upside-down (180 deg roll about X) per
  the real physical mount. The URDF's +/-90 deg roll values were
  consistent with the physical robot's "one inverted" config.
- Webots' rotating-lidar type can't simulate the real MID-360's
  Risley-prism asymmetric FOV; sticking to symmetric ±15 deg is
  pragmatic.

Density tuned for Webots (real device is ~200k pts/s non-repetitive;
sim is rotating-multilayer):
- horizontalResolution 900, layers 16 -> ~144k pts/s per lidar.
- Earlier 1800x64 push lagged the system.

Dual-lidar merger (scripts/livox_merger.py):
- Subscribes to both lidar topics, applies the known static transform
  (Rx(180 deg) + 7 cm Z) to bottom points, concatenates, publishes
  /livox/lidar at frame=livox_frame.
- Drops NaN points (Webots returns NaN for misses).
- KISS-ICP then ingests one cloud combining both lidars.

TF cleanup:
- rove_driver.py: new publish_odom_tf property (default false). Stops
  the wheel-integrated odom->base_link TF that was racing SLAM's
  TF and making the position appear to jump. The /odom topic
  still publishes for downstream fusion.

Co-Authored-By: Claude Opus 4.7 <noreply@anthropic.com>

File: src/rove_sim_webots/urdf/rove_webots.urdf (robot description, URDF)
Before this commit: robot rove, 3 links, 2 joints
Links:
- removed link camera_link
- removed link livox_frame
- added link Core
Joints:
- removed joint camera_joint
- removed joint livox_joint
- added joint base_to_core: type fixed, parent base_link, child Core, origin xyz=0 0 0 rpy=0 0 0
